Commit message: change bounce

File: hockey_robot_description/urdf/hockey_robot.xacro (robot description, xacro)
@@ -8,4 +8,8 @@
   <xacro:property name="camera_height" value="1.5" /> <!-- Link 3 -->
   <xacro:property name="camera_link" value="0.05" /> <!-- Size of square 'camera' box -->
+  <xacro:property name="sonar_length" value="0.07" />
+  <xacro:property name="sonar_width" value="0.01" />
+  <xacro:property name="sonar_height" value="0.02" />
+  <xacro:property name="sonar_link" value="0.1" />
   <xacro:property name="pusher_height" value="0.02" /> <!-- Space btw top of beam and the each joint -->
   <xacro:property name="pusher_radius" value="0.045" />
@@ -23,5 +27,5 @@
     <visual>
       <geometry>
-        <mesh filename="package://hockey_robot_description/meshes/hockeytable.dae"/>
+        <mesh filename="package://hockey_robot_description/meshes/hockeytablev2.dae"/>
       </geometry>
       <origin rpy="0 0 0" xyz="-0.46 -0.7 -0.8"/>
@@ -30,8 +34,7 @@
     <collision>
       <geometry>
-        <mesh filename="package://hockey_robot_description/meshes/hockeytable.dae"/>
+        <mesh filename="package://hockey_robot_description/meshes/hockeytablev2.dae"/>
       </geometry>
       <origin rpy="0 0 0" xyz="-0.46 -0.7 -0.8"/>
-      <contact_coefficients mu="0" resitution="0" k_p="100" k_d="0" />
     </collision>
     <inertial>
@@ -45,11 +48,11 @@
       <origin xyz="0 0 0" rpy="0 0 0"/>
       <geometry>
-	<box size="${camera_link} ${camera_link} ${camera_link}"/>
-      </geometry>
-    </collision>
-    <visual>
-      <origin xyz="0 0 0" rpy="0 0 0"/>
-      <geometry>
-	<box size="${camera_link} ${camera_link} ${camera_link}"/>
+	      <box size="${camera_link} ${camera_link} ${camera_link}"/>
+      </geometry>
+    </collision>
+    <visual>
+      <origin xyz="0 0 0" rpy="0 0 0"/>
+      <geometry>
+	      <box size="${camera_link} ${camera_link} ${camera_link}"/>
       </geometry>
       <material name="white"/>
@@ -67,4 +70,59 @@
     <parent link="base_link"/>
     <child link="camera_link"/>
+  </joint>
+  <!-- Sonar -->
+  <link name="sonar_1">
+    <collision>
+      <origin xyz="0 0 0" rpy="0 0 0"/>
+      <geometry>
+	      <box size="${sonar_width} ${sonar_length} ${sonar_height}"/>
+      </geometry>
+    </collision>
+    <visual>
+      <origin xyz="0 0 0" rpy="0 0 0"/>
+      <geometry>
+	      <box size="${sonar_width} ${sonar_length} ${sonar_height}"/>
+      </geometry>
+      <material name="blue"/>
+    </visual>
+    <inertial>
+      <mass value="1e-5" />
+      <origin xyz="0 0 0" rpy="0 0 0"/>
+      <inertia ixx="1e-6" ixy="0" ixz="0" iyy="1e-6" iyz="0" izz="1e-6" />
+    </inertial>
+  </link>
+  <joint name="sonar_1_joint" type="fixed">
+    <axis xyz="0 0 0" />
+    <!--rigin xyz="0 1 ${height3 - axel_offset*2}" rpy="0 0 0"/-->
+    <origin xyz="-0.15 -0.95 ${sonar_height/2}" rpy="0 0 0"/>
+    <parent link="base_link"/>
+    <child link="sonar_1"/>
+  </joint>
+  <link name="sonar_2">
+    <collision>
+      <origin xyz="0 0 0" rpy="0 0 0"/>
+      <geometry>
+	      <box size="${sonar_width} ${sonar_length} ${sonar_height}"/>
+      </geometry>
+    </collision>
+    <visual>
+      <origin xyz="0 0 0" rpy="0 0 0"/>
+      <geometry>
+	      <box size="${sonar_width} ${sonar_length} ${sonar_height}"/>
+      </geometry>
+      <material name="blue"/>
+    </visual>
+    <inertial>
+      <mass value="1e-5" />
+      <origin xyz="0 0 0" rpy="0 0 0"/>
+      <inertia ixx="1e-6" ixy="0" ixz="0" iyy="1e-6" iyz="0" izz="1e-6" />
+    </inertial>
+  </link>
+  <joint name="sonar_2_joint" type="fixed">
+    <axis xyz="0 0 0" />
+    <!--rigin xyz="0 1 ${height3 - axel_offset*2}" rpy="0 0 0"/-->
+    <origin xyz="0.15 0.95 ${sonar_height/2}" rpy="0 0 ${pi}"/>
+    <parent link="base_link"/>
+    <child link="sonar_2"/>
   </joint>
   <!-- generate an optical frame http://www.ros.org/reps/rep-0103.html#suffix-frames
@@ -199,5 +257,5 @@
     </actuator>
   </transmission>
-    <transmission name="tran3">
+  <transmission name="tran3">
     <type>transmission_interface/SimpleTransmission</type>
     <joint name="base_to_horizon_track_2">

Commit message: update

File: hockey_robot_description/urdf/hockey_robot.xacro (robot description, xacro)
@@ -140,5 +140,5 @@
     <visual>
       <geometry>
-        <box size="${width} 0.05 0.01"/>
+        <box size="${width} 0.01 0.01"/>
       </geometry>
       <origin rpy="0 0 0" xyz="0 0 0"/>
@@ -190,5 +190,5 @@
     <visual>
       <geometry>
-        <box size="${width} 0.05 0.01"/>
+        <box size="${width} 0.01 0.01"/>
       </geometry>
       <origin rpy="0 0 0" xyz="0 0 0"/>

Commit message: update

File: hockey_robot_description/urdf/hockey_robot.xacro (robot description, xacro)
@@ -140,5 +140,5 @@
     <visual>
       <geometry>
-        <box size="${width} 0.01 0.01"/>
+        <box size="${width} 0 0"/>
       </geometry>
       <origin rpy="0 0 0" xyz="0 0 0"/>
@@ -174,4 +174,7 @@
         <cylinder length="${pusher_height}" radius="${pusher_radius}"/>
       </geometry>
+      <surface>
+        <bounce restitution_coefficient="1.0" threshold="0.01"/>
+      </surface>
     </collision>
     <inertial>
@@ -190,5 +193,5 @@
     <visual>
       <geometry>
-        <box size="${width} 0.01 0.01"/>
+        <box size="${width} 0 0"/>
       </geometry>
       <origin rpy="0 0 0" xyz="0 0 0"/>
@@ -210,5 +213,5 @@
     <parent link="base_link"/>
     <child link="horizon_track_2"/>
-    <limit effort="1000.0" lower="0" upper="${tackers_radius}" velocity="0.5"/>
+    <limit effort="1000.0" lower="0" upper="${tackers_radius}" velocity="1"/>
     <origin xyz="0 ${tackers_radius} ${tackers_height}" rpy="0 0 ${pi}"/>
   </joint>
@@ -234,7 +237,14 @@
     <parent link="horizon_track_2"/>
     <child link="pusher_2"/>
-    <limit effort="1000.0" lower="-0.5" upper="0.5" velocity="0.5"/>
+    <limit effort="1000.0" lower="-0.5" upper="0.5" velocity="1"/>
     <origin xyz="0 0 -${tackers_height-pusher_height/2}"/>
   </joint>
+  <!-- <joint name="base_to_horizon_track_2_2" type="prismatic">
+    <axis xyz="0 1 0"/>
+    <parent link="base_link"/>
+    <child link="horizon_track_2"/>
+    <limit effort="1000.0" lower="0" upper="${tackers_radius}" velocity="0.5"/>
+    <origin xyz="0 ${tackers_radius} ${tackers_height}" rpy="0 0 ${pi}"/>
+  </joint> -->
   <transmission name="tran1">
     <type>transmission_interface/SimpleTransmission</type>
@@ -277,3 +287,13 @@
     </actuator>
   </transmission>
+  <!-- <transmission name="tran5">
+    <type>transmission_interface/SimpleTransmission</type>
+    <joint name="base_to_horizon_track_2_2">
+      <hardwareInterface>EffortJointInterface</hardwareInterface>
+    </joint>
+    <actuator name="motor5">
+      <hardwareInterface>EffortJointInterface</hardwareInterface>
+      <mechanicalReduction>1</mechanicalReduction>
+    </actuator>
+  </transmission> -->
 </robot>

Commit message: update

File: hockey_robot_description/urdf/hockey_robot.xacro (robot description, xacro)
@@ -13,5 +13,5 @@
   <xacro:property name="sonar_link" value="0.1" />
   <xacro:property name="pusher_height" value="0.02" /> <!-- Space btw top of beam and the each joint -->
-  <xacro:property name="pusher_radius" value="0.045" />
+  <xacro:property name="pusher_radius" value="0.04" />
   <!-- Import all Gazebo-customization elements, including Gazebo colors -->
   <xacro:include filename="$(find hockey_robot_description)/urdf/hockey_robot.gazebo" />
@@ -27,5 +27,5 @@
     <visual>
       <geometry>
-        <mesh filename="package://hockey_robot_description/meshes/hockeytablev2.dae"/>
+        <mesh filename="package://hockey_robot_description/meshes/hockeytablev4.dae"/>
       </geometry>
       <origin rpy="0 0 0" xyz="-0.46 -0.7 -0.8"/>
@@ -34,5 +34,5 @@
     <collision>
       <geometry>
-        <mesh filename="package://hockey_robot_description/meshes/hockeytablev2.dae"/>
+        <mesh filename="package://hockey_robot_description/meshes/hockeytablev4.dae"/>
       </geometry>
       <origin rpy="0 0 0" xyz="-0.46 -0.7 -0.8"/>
@@ -95,5 +95,5 @@
     <axis xyz="0 0 0" />
     <!--rigin xyz="0 1 ${height3 - axel_offset*2}" rpy="0 0 0"/-->
-    <origin xyz="-0.15 -0.95 ${sonar_height/2}" rpy="0 0 0"/>
+    <origin xyz="-0.26 -0.95 ${sonar_height/2}" rpy="0 0 0"/>
     <parent link="base_link"/>
     <child link="sonar_1"/>
@@ -122,5 +122,5 @@
     <axis xyz="0 0 0" />
     <!--rigin xyz="0 1 ${height3 - axel_offset*2}" rpy="0 0 0"/-->
-    <origin xyz="0.15 0.95 ${sonar_height/2}" rpy="0 0 ${pi}"/>
+    <origin xyz="0.26 0.95 ${sonar_height/2}" rpy="0 0 ${pi}"/>
     <parent link="base_link"/>
     <child link="sonar_2"/>
@@ -219,5 +219,5 @@
     <visual>
       <geometry>
-        <cylinder length="0.02" radius="0.045"/>
+        <cylinder length="0.02" radius="${pusher_radius}"/>
       </geometry>
       <material name="black"/>
@@ -225,5 +225,5 @@
     <collision>
       <geometry>
-        <cylinder length="0.02" radius="0.045"/>
+        <cylinder length="0.02" radius="${pusher_radius}"/>
       </geometry>
     </collision>
